Commit message: Updated camera URDFs

File: rasprover_description/urdf/dons_rasprover_gazebo.urdf (robot description, URDF)
Before this commit: robot rasprover, 10 links, 9 joints
Links:
- link camera_link: geometry collision cylinder length=0.020 radius=0.015; visual mesh filename=package://rasprover_description/meshes/pt_camera_link.stl
Joints:
- joint camera_joint: origin xyz=0.065 0.0 0.086 rpy=0 1.55 0 -> xyz=0.050 0.0 0.086 rpy=0 1.55 0
